File: uSD_extender_female.brd (EAGLE design)
At the start: 15.6 x 24.9 mm, 5 parts

Commit message: Update uSD_extender_female.brd
Parts:
- removed U$3, U$4, U$5: SMALL_WIRE_HOLE, Dean:SMALL_WIRE_HOLE
- U$1: value MICROSD -> DEAN_MICROSD; device Dean:MICROSD -> uSD_extender_female:DEAN_MICROSD
Connections:
- removed net N$7: U$1.CD1, U$4.P$1
- removed net N$8: U$1.CD2, U$3.P$1
- net GND: no longer U$5.P$1
Routing:
- net GND: track 19.4 -> 0.00 mm
- net N$8: track 11.9 -> 0.00 mm, vias 1 -> 0
- net N$7: track 5.38 -> 0.00 mm
Other:
- board size 15.6 x 24.9 mm -> 24.8 x 25.4 mm
- board text removed: "CD"
- board text removed: "GND"
